File: Project/Board_CAN_Connector.sch (KiCad schematic (older format))
At the start: 3 parts, among them J19 649006227222

Commit message: last changes
Changed lines of the file:
@@
 $Descr A4 11693 8268
 encoding utf-8
-Sheet 9 22
+Sheet 15 22
 Title ""
 Date ""
@@
 AR Path="/5FEFC7D4/5FF30BE7/5FF0A0A5" Ref="J26"  Part="1"
 AR Path="/5FEFC7D4/601F2198/5FF0A0A5" Ref="J30"  Part="1"
-F 0 "J25" H 9750 2750 60  0000 C CNN
+F 0 "J20" H 9750 2750 60  0000 C CNN
 F 1 "649006227222" H 9750 2650 60  0000 C CNN
 F 2 "Connectors:649006227222" H 9750 1350 60  0001 C CNN
@@
 AR Path="/5FEFC7D4/5FF30A38/600C1D05" Ref="C35"  Part="1"
 AR Path="/5FEFC7D4/5FF3099D/600C1D05" Ref="C37"  Part="1"
-F 0 "C17" H 4800 1948 60  0000 C CNN
+F 0 "C39" H 4800 1948 60  0000 C CNN
 F 1 "885012107015" H 4800 1350 60  0001 C CNN
 F 2 "Capacitors:C0805" H 4800 750 60  0001 C CNN
@@
 AR Path="/5FEFC7D4/5FF3099D/600CFE9E" Ref="C26"  Part="1"
 AR Path="/5FEFC7D4/5FF30935/600CFE9E" Ref="C27"  Part="1"
-F 0 "C19" V 4955 1905 60  0000 L CNN
+F 0 "C27" V 4955 1905 60  0000 L CNN
 F 1 "885012207098" H 5000 1450 60  0001 C CNN
 F 2 "Capacitors:C0805" H 5000 850 60  0001 C CNN

Commit message: Code review changes
Changed lines of the file:
@@
 $Descr A4 11693 8268
 encoding utf-8
-Sheet 15 22
+Sheet 8 23
 Title ""
 Date ""
@@
 AR Path="/5FEFC7D4/5FF30BE7/5FF077E8" Ref="#PWR064"  Part="1"
 AR Path="/5FEFC7D4/601F2198/5FF077E8" Ref="#PWR041"  Part="1"
-F 0 "#PWR034" H 6450 2280 50  0001 C CNN
+F 0 "#PWR064" H 6450 2280 50  0001 C CNN
 F 1 "DGND" H 6450 2350 50  0000 C CNN
 F 2 "" H 6450 2550 60  0000 C CNN
@@
 AR Path="/5FEFC7D4/5FF30BE7/5FF0A0A5" Ref="J26"  Part="1"
 AR Path="/5FEFC7D4/601F2198/5FF0A0A5" Ref="J30"  Part="1"
-F 0 "J20" H 9750 2750 60  0000 C CNN
+F 0 "J26" H 9750 2750 60  0000 C CNN
 F 1 "649006227222" H 9750 2650 60  0000 C CNN
 F 2 "Connectors:649006227222" H 9750 1350 60  0001 C CNN
@@
 AR Path="/5FEFC7D4/5FF3099D/5FF27778" Ref="#PWR094"  Part="1"
 AR Path="/5FEFC7D4/5FF30935/5FF27778" Ref="#PWR096"  Part="1"
-F 0 "#PWR096" H 10050 1780 50  0001 C CNN
+F 0 "#PWR082" H 10050 1780 50  0001 C CNN
 F 1 "DGND" V 10050 1650 50  0000 L CNN
 F 2 "" H 10050 2050 60  0000 C CNN
@@
 AR Path="/5FEFC7D4/5FF3099D/5FF27EA7" Ref="#PWR093"  Part="1"
 AR Path="/5FEFC7D4/5FF30935/5FF27EA7" Ref="#PWR095"  Part="1"
-F 0 "#PWR095" H 9450 1780 50  0001 C CNN
+F 0 "#PWR081" H 9450 1780 50  0001 C CNN
 F 1 "DGND" V 9450 1650 50  0000 L CNN
 F 2 "" H 9450 2050 60  0000 C CNN
@@
 AR Path="/5FEFC7D4/5FF30A38/600C1D05" Ref="C35"  Part="1"
 AR Path="/5FEFC7D4/5FF3099D/600C1D05" Ref="C37"  Part="1"
-F 0 "C39" H 4800 1948 60  0000 C CNN
+F 0 "C5" H 4800 1948 60  0000 C CNN
 F 1 "885012107015" H 4800 1350 60  0001 C CNN
 F 2 "Capacitors:C0805" H 4800 750 60  0001 C CNN
@@
 AR Path="/5FEFC7D4/5FF3099D/600CFE9E" Ref="C26"  Part="1"
 AR Path="/5FEFC7D4/5FF30935/600CFE9E" Ref="C27"  Part="1"
-F 0 "C27" V 4955 1905 60  0000 L CNN
+F 0 "C15" V 4955 1905 60  0000 L CNN
 F 1 "885012207098" H 5000 1450 60  0001 C CNN
 F 2 "Capacitors:C0805" H 5000 850 60  0001 C CNN
@@
 AR Path="/5FEFC7D4/5FF3099D/600D3910" Ref="#PWR0118"  Part="1"
 AR Path="/5FEFC7D4/5FF30935/600D3910" Ref="#PWR0120"  Part="1"
-F 0 "#PWR0120" H 5050 1830 50  0001 C CNN
+F 0 "#PWR0101" H 5050 1830 50  0001 C CNN
 F 1 "DGND" H 5100 1850 50  0000 C CNN
 F 2 "" H 5050 2100 60  0000 C CNN
@@
 AR Path="/5FEFC7D4/5FF3099D/600D3D6B" Ref="#PWR0119"  Part="1"
 AR Path="/5FEFC7D4/5FF30935/600D3D6B" Ref="#PWR0121"  Part="1"
-F 0 "#PWR0121" H 4850 1830 50  0001 C CNN
+F 0 "#PWR0102" H 4850 1830 50  0001 C CNN
 F 1 "DGND" H 4800 1850 50  0000 C CNN
 F 2 "" H 4850 2100 60  0000 C CNN
