File: Project/CAN_Connectors.sch (KiCad schematic (older format))
At the start: 14 parts, among them J30 649006227222, U8 SN65HVD232DR

Commit message: Code review changes
Connections:
- net labels removed: CAN_N, CAN_P, CAN_PWR
- wire segments 127 -> 104
- no-connect marks 2 -> 3
