File: Project/CurrentSense12V.sch (KiCad schematic (older format))
At the start: 8 parts, among them U6 LTC2992IMS_PBF

Commit message: last changes
Changed lines of the file:
@@
 $Descr A4 11693 8268
 encoding utf-8
-Sheet 18 22
+Sheet 16 22
 Title ""
 Date ""
@@
 AR Path="/5FEFC7D4/5FF307B6/5FEFFCB2" Ref="#PWR067"  Part="1"
 AR Path="/5FEFC7D4/5FF307BE/5FEFFCB2" Ref="#PWR076"  Part="1"
-F 0 "#PWR076" H 6450 4280 50  0001 C CNN
+F 0 "#PWR048" H 6450 4280 50  0001 C CNN
 F 1 "DGND" H 6450 4300 50  0000 C CNN
 F 2 "" H 6450 4550 60  0000 C CNN
@@
 AR Path="/5FEFC7D4/5FF307B6/5FF0113A" Ref="R31"  Part="1"
 AR Path="/5FEFC7D4/5FF307BE/5FF0113A" Ref="R37"  Part="1"
-F 0 "R37" V 3941 2342 60  0000 R CNN
+F 0 "R19" V 3941 2342 60  0000 R CNN
 F 1 "ERJ-6LWFR005V" H 3900 2100 50  0001 C CNN
 F 2 "Resistors:R0805" H 3900 1500 30  0001 C CNN
@@
 AR Path="/5FEFC7D4/5FF307B6/5FF02241" Ref="R32"  Part="1"
 AR Path="/5FEFC7D4/5FF307BE/5FF02241" Ref="R38"  Part="1"
-F 0 "R38" V 3759 3058 60  0000 L CNN
+F 0 "R20" V 3759 3058 60  0000 L CNN
 F 1 "ERJ-6LWFR005V" H 3900 2700 50  0001 C CNN
 F 2 "Resistors:R0805" H 3900 2100 30  0001 C CNN
@@
 AR Path="/5FEFC7D4/5FF307BE/5FEFE842" Ref="U11"  Part="1"
 AR Path="/5FEFE842" Ref="U6"  Part="1"
-F 0 "U11" H 5550 6689 60  0000 C CNN
+F 0 "U6" H 5550 6689 60  0000 C CNN
 F 1 "LTC2992IMS_PBF" H 5550 6583 60  0000 C CNN
 F 2 "IC:AnalogDevices_16-MSOP" H 5560 3560 60  0001 C CNN
@@
 AR Path="/5FEFC7D4/5FF307B6/5FEE539C" Ref="R34"  Part="1"
 AR Path="/5FEFC7D4/5FF307BE/5FEE539C" Ref="R40"  Part="1"
-F 0 "R40" V 8405 3058 60  0000 L CNN
+F 0 "R22" V 8405 3058 60  0000 L CNN
 F 1 "0hms_0.5W" H 8450 2700 50  0001 C CNN
 F 2 "Resistors:R0805" H 8450 2100 30  0001 C CNN
@@
 AR Path="/5FEFC7D4/5FF307B6/5FEE7D07" Ref="R33"  Part="1"
 AR Path="/5FEFC7D4/5FF307BE/5FEE7D07" Ref="R39"  Part="1"
-F 0 "R39" V 8495 2342 60  0000 R CNN
+F 0 "R21" V 8495 2342 60  0000 R CNN
 F 1 "0hms_0.5W" H 8450 2100 50  0001 C CNN
 F 2 "Resistors:R0805" H 8450 1500 30  0001 C CNN
@@
 AR Path="/5FEFC7D4/5FF307B6/5FEED535" Ref="R36"  Part="1"
 AR Path="/5FEFC7D4/5FF307BE/5FEED535" Ref="R42"  Part="1"
-F 0 "R42" V 9205 3058 60  0000 L CNN
+F 0 "R24" V 9205 3058 60  0000 L CNN
 F 1 "0hms_0.5W" H 9250 2700 50  0001 C CNN
 F 2 "Resistors:R0805" H 9250 2100 30  0001 C CNN
@@
 AR Path="/5FEFC7D4/5FF307B6/5FEED542" Ref="R35"  Part="1"
 AR Path="/5FEFC7D4/5FF307BE/5FEED542" Ref="R41"  Part="1"
-F 0 "R41" V 9295 2342 60  0000 R CNN
+F 0 "R23" V 9295 2342 60  0000 R CNN
 F 1 "0hms_0.5W" H 9250 2100 50  0001 C CNN
 F 2 "Resistors:R0805" H 9250 1500 30  0001 C CNN
@@
 AR Path="/5FEFC7D4/5FF307B6/5FEF5663" Ref="#PWR071"  Part="1"
 AR Path="/5FEFC7D4/5FF307BE/5FEF5663" Ref="#PWR078"  Part="1"
-F 0 "#PWR078" H 8450 3130 50  0001 C CNN
+F 0 "#PWR052" H 8450 3130 50  0001 C CNN
 F 1 "DGND" H 8450 3150 50  0000 C CNN
 F 2 "" H 8450 3400 60  0000 C CNN
@@
 AR Path="/5FEFC7D4/5FF307B6/5FEF5B01" Ref="#PWR073"  Part="1"
 AR Path="/5FEFC7D4/5FF307BE/5FEF5B01" Ref="#PWR080"  Part="1"
-F 0 "#PWR080" H 9250 3130 50  0001 C CNN
+F 0 "#PWR055" H 9250 3130 50  0001 C CNN
 F 1 "DGND" H 9250 3150 50  0000 C CNN
 F 2 "" H 9250 3400 60  0000 C CNN
@@
 AR Path="/5FEFC7D4/5FF307B6/5FF22874" Ref="#PWR016"  Part="1"
 AR Path="/5FEFC7D4/5FF307BE/5FF22874" Ref="#PWR017"  Part="1"
-F 0 "#PWR017" H 6450 1800 50  0001 C CNN
+F 0 "#PWR014" H 6450 1800 50  0001 C CNN
 F 1 "CAN_PWR" H 6450 2123 50  0000 C CNN
 F 2 "" H 6450 1950 60  0000 C CNN
@@
 AR Path="/5FEFC7D4/5FF307B6/5FF25A62" Ref="C3"  Part="1"
 AR Path="/5FEFC7D4/5FF307BE/5FF25A62" Ref="C4"  Part="1"
-F 0 "C4" V 6355 2805 60  0000 L CNN
+F 0 "C1" V 6355 2805 60  0000 L CNN
 F 1 "885012207098" H 6400 2350 60  0001 C CNN
 F 2 "Capacitors:C0805" H 6400 1750 60  0001 C CNN
@@
 AR Path="/5FEFC7D4/5FF307B6/5FFF8ADE" Ref="#FLG0103"  Part="1"
 AR Path="/5FEFC7D4/5FF307BE/5FFF8ADE" Ref="#FLG0104"  Part="1"
-F 0 "#FLG0104" H 6850 2200 60  0001 C CNN
+F 0 "#FLG0101" H 6850 2200 60  0001 C CNN
 F 1 "PWR_FLAG" V 6850 2478 30  0000 L CNN
 F 2 "" H 6850 2300 60  0000 C CNN

Commit message: Code review changes
Parts:
- removed R21, R22, R23, R24: 0hms_0.5W, Resistors:R0805, symbol Resistors:0hms_0.5W
Connections:
- wire segments 35 -> 36
- no-connect marks 4 -> 0
Other:
- note removed: "Only Solder Necessary"
