File: Project/HW_Testbench.kicad_pcb (KiCad board)
At the start: 2 copper layers, 144.8 x 88.9 mm, 161 parts, among them J1 61900611121, J107 Header_Male_Pin_2.54mm_1X2_,_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, J15 Header_Male_Pin_2.54mm_1X3_,_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, J16 Header_Male_Pin_2.54mm_1X3_,_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, J17 Header_Male_Pin_2.54mm_1X3_,_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, J18 Header_Male_Pin_2.54mm_1X3_,_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, J19 649006227222, J2 61900611121, J20 649006227222, J202 Header_Male_Pin_2.54mm_1X3_,_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, J21 649006227222, J22 649006227222, J23 649006227222, J24 649006227222, J25 649006227222, J26 649006227222, J27 1935161, J28 61900611121, J29 61900611121, J3 61900611121, J30 649006227222, J301 Header_Male_Pin_2.54mm_1X2_,_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, J4 61900611121, J5 61900611121, J6 61900611121, J7 61900611121, J8 61900611121, J9 61900611121, SW201 PTS645SM43SMTR92, SW202 PTS645SM43SMTR92, U1 TMUX1208PWR, U10 LTC2992IMS_PBF, U11 LTC2992IMS_PBF, U12 STLINK-V3MODS, U2 TMUX1208PWR, U201 STM32F446RE, U3 TMUX1208PWR, U301 OKI-78SR-5_1.5-W36H-C, U302 AZ1117IH-3.3TRG1, U4 TMUX1208PWR, U6 LTC2992IMS_PBF, U7 SN65HVD232DR, U8 SN65HVD232DR, U9 LTC2992IMS_PBF

Commit message: last changes
Routing:
- net DGND: track 206.6 -> 211.8 mm, vias 36 -> 37
Changed lines of the file:
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@@
     (thickness 1.6)
     (drawings 39)
-    (tracks 2046)
+    (tracks 2050)
     (zones 0)
     (modules 161)
@@
   (segment (start 34.1884 32.1564) (end 33.8328 31.8008) (width 0.254) (layer F.Cu) (net 1))
   (segment (start 35.2552 32.1564) (end 34.1884 32.1564) (width 0.254) (layer F.Cu) (net 1))
+  (via (at 55.88 84.0232) (size 0.8) (drill 0.4) (layers F.Cu B.Cu) (net 1))
+  (segment (start 55.88 80.433) (end 55.88 84.0232) (width 0.254) (layer F.Cu) (net 1))
+  (segment (start 55.461 80.014) (end 55.88 80.433) (width 0.254) (layer F.Cu) (net 1))
+  (segment (start 54.482 80.014) (end 55.461 80.014) (width 0.254) (layer F.Cu) (net 1))
   (via (at 42.7736 58.7756) (size 0.8) (drill 0.4) (layers F.Cu B.Cu) (net 2))
   (via (at 45.2628 58.7756) (size 0.8) (drill 0.4) (layers F.Cu B.Cu) (net 2))

Commit message: Code review changes
Parts:
- removed C1, C2, C3, C4: 885012207098, Capacitors:C0805
- removed R19, R20, R25, R26, R31, R32, R37, R38: ERJ-6LWFR005V, Resistors:R0805
- removed R21, R22, R23, R24, R27, R28, R29, R30, R33, R34, R35, R36, R39, R40, R41, R42: 0hms_0.5W, Resistors:R0805
- removed U10, U11, U6, U9: LTC2992IMS_PBF, IC:AnalogDevices_16-MSOP
- added C1701: 885012207098, Capacitors:C0805, B.Cu at (45.9, 33.7)
- added C1801: 885012207098, Capacitors:C0805, B.Cu at (132.3, 81.9)
- added C1901: 885012207098, Capacitors:C0805, B.Cu at (128.0, 34.1)
- added C2001: 885012207098, Capacitors:C0805, B.Cu at (55.9, 80.5)
- added R1601: RC0805JR-070RL, Resistors:R0805, B.Cu at (53.1, 30.8)
- added R1602: RC0805JR-070RL, Resistors:R0805, B.Cu at (56.4, 31.4)
- added R1603: RC0805JR-070RL, Resistors:R0805, B.Cu at (126.5, 36.5)
- added R1604: RC0805JR-070RL, Resistors:R0805, B.Cu at (124.5, 39.1)
- added R1605: RC0805JR-070RL, Resistors:R0805, B.Cu at (47.9, 31.5)
- added R1606: RC0805JR-070RL, Resistors:R0805, B.Cu at (50.0, 29.0)
- added R1607: RC0805JR-070RL, Resistors:R0805, B.Cu at (119.8, 36.4)
- added R1608: RC0805JR-070RL, Resistors:R0805, B.Cu at (121.8, 39.1)
- added R1609: RC0805JR-070RL, Resistors:R0805, B.Cu at (126.2, 72.1)
- added R1610: RC0805JR-070RL, Resistors:R0805, B.Cu at (128.3, 69.3)
- added R1611: RC0805JR-070RL, Resistors:R0805, B.Cu at (56.4, 76.2)
- added R1612: RC0805JR-070RL, Resistors:R0805, B.Cu at (58.4, 73.5)
- added R1613: RC0805JR-070RL, Resistors:R0805, B.Cu at (132.4, 76.9)
- added R1614: RC0805JR-070RL, Resistors:R0805, B.Cu at (130.3, 74.1)
- added R1615: RC0805JR-070RL, Resistors:R0805, B.Cu at (63.6, 77.1)
- added R1616: RC0805JR-070RL, Resistors:R0805, B.Cu at (61.5, 74.4)
- added R1701: ERJ-6LWFR005V, Resistors:R0805, F.Cu at (50.9, 30.0)
- added R1702: ERJ-6LWFR005V, Resistors:R0805, F.Cu at (62.6, 32.1)
- added R1801: ERJ-6LWFR005V, Resistors:R0805, F.Cu at (131.8, 82.8)
- added R1802: ERJ-6LWFR005V, Resistors:R0805, F.Cu at (120.8, 80.7)
- added R1901: ERJ-6LWFR005V, Resistors:R0805, F.Cu at (120.5, 30.0)
- added R1902: ERJ-6LWFR005V, Resistors:R0805, F.Cu at (132.1, 32.1)
- added R2001: ERJ-6LWFR005V, Resistors:R0805, F.Cu at (62.0, 82.8)
- added R2002: ERJ-6LWFR005V, Resistors:R0805, F.Cu at (50.8, 80.7)
- added U1701: LTC2992IMS_PBF, IC:AnalogDevices_16-MSOP, F.Cu at (56.6, 32.5)
- added U1801: LTC2992IMS_PBF, IC:AnalogDevices_16-MSOP, F.Cu at (126.4, 80.3)
- added U1901: LTC2992IMS_PBF, IC:AnalogDevices_16-MSOP, F.Cu at (126.2, 32.5)
- added U2001: LTC2992IMS_PBF, IC:AnalogDevices_16-MSOP, F.Cu at (56.7, 80.3)
Connections:
- J30 pad 5: CAN_PWR -> Net-(J30-Pad5)
Routing:
- net DGND: track 211.8 -> 238.3 mm, vias 37 -> 40
- net /CAN_Connectors/CurrentSense_3/INTVcc: track 23.3 -> 0.00 mm, vias 2 -> 0
- net /CAN_Connectors/CurrentSense/sheet60485D36/INTVcc: track 0.00 -> 23.3 mm, vias 0 -> 2
- net /CAN_Connectors/CurrentSense_2/INTVcc: track 19.9 -> 0.00 mm, vias 1 -> 0
- net /CAN_Connectors/CurrentSense/sheet60485D37/INTVcc: track 0.00 -> 19.9 mm, vias 0 -> 1
- net /CAN_Connectors/CurrentSense_4/INTVcc: track 18.9 -> 0.00 mm, vias 1 -> 0
- net /CAN_Connectors/CurrentSense/sheet60485D38/INTVcc: track 0.00 -> 18.9 mm, vias 0 -> 1
- net /CAN_Connectors/CurrentSense_1/INTVcc: track 18.6 -> 0.00 mm, vias 1 -> 0
- net /CAN_Connectors/CurrentSense/sheet60485D35/INTVcc: track 0.00 -> 18.6 mm, vias 0 -> 1
- net /CAN_Connectors/CurrentSense_3/I2C_ADR0: track 12.9 -> 0.00 mm, vias 1 -> 0
- net /CAN_Connectors/CurrentSense/sheet60485D36/I2C_ADR0: track 0.00 -> 12.9 mm, vias 0 -> 1
- net /CAN_Connectors/CurrentSense_2/I2C_ADR0: track 8.75 -> 0.00 mm, vias 1 -> 0
- net /CAN_Connectors/CurrentSense/sheet60485D37/I2C_ADR0: track 0.00 -> 8.75 mm, vias 0 -> 1
- net /CAN_Connectors/CurrentSense_1/I2C_ADR0: track 8.71 -> 0.00 mm, vias 1 -> 0
- net /CAN_Connectors/CurrentSense/sheet60485D35/I2C_ADR0: track 0.00 -> 8.71 mm, vias 0 -> 1
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