File: Project/HW_Testbench.sch (KiCad schematic (older format))
At the start: 4 parts, among them J1 61900611121, J107 Header_Male_Pin_2.54mm_1X2_,_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, J2 61900611121, J3 61900611121

Commit message: Code review changes
Other:
- note added: "GND Testpoint"
Changed lines of the file:
@@
 $Descr USLetter 11000 8500
 encoding utf-8
-Sheet 1 22
+Sheet 1 23
 Title ""
 Date ""
@@
 NoConn ~ 8800 2750
 NoConn ~ 8800 3450
+Text Notes 700  1000 0    50   ~ 0
+GND Testpoint
 Wire Bus Line
 	8200 3000 8200 3250
